File: Design/Sensing/sensor/kicad_simulations/sensor/sensor.kicad_pcb (KiCad board)
At the start: 2 copper layers, 61.2 x 37.5 mm, 38 parts, among them J1 Conn_01x02_Pin, J10 Conn_01x02_Pin, J11 Conn_01x02_Pin, J12 Conn_01x02_Pin, J13 Conn_01x02_Pin, J14 Conn_01x01_Pin, J15 Conn_01x01_Pin, J16 Conn_01x02_Pin, J17 Conn_01x02_Pin, J2 Conn_01x02_Pin, J3 Conn_02x14_Counter_Clockwise, J5 L_S_B, J6 Conn_01x01_Pin, J7 Conn_01x02_Pin, J8 Conn_01x02_Pin, J9 Conn_01x02_Pin, Q1 MMBT5551L, Q2 MMBT5551L, Q3 MMBT5551L, U1 LM324, U2 TSSP58038, U3 TSSP58038, U4 TSSP58038

Commit message: IR change
Parts:
- removed D5: TSAL4400, LED_THT:LED_D3.0mm_Horizontal_O1.27mm_Z2.0mm_IRBlack
- added D2: IR204A, LED_THT:LED_D3.0mm_Horizontal_O1.27mm_Z2.0mm_IRBlack, F.Cu at (119.9, 91.1)
- D1, D3: value TSAL4400 -> IR204A
- R1, R2, R3, R5, R6: footprint Resistor_SMD:R_1206_3216Metric -> Resistor_SMD:R_0805_2012Metric
- moved D1 41.5 mm to (161.3, 92.3), turned to 135 degrees
- moved D3 21.7 mm to (140.8, 85.8), turned to 180 degrees
Connections:
- R2 pad 2: Net-(D1-K) -> Net-(D2-K)
- R5 pad 2: Net-(D3-K) -> Net-(D1-K)
- R6 pad 2: Net-(D5-K) -> Net-(D3-K)
Routing:
- net Net-(D2-K): track 0.00 -> 8.05 mm
- net Net-(D3-K): track 13.4 -> 6.10 mm, vias 2 -> 0
- net Net-(D5-K): track 6.10 -> 0.00 mm
- net Net-(D1-K): track 8.05 -> 13.4 mm, vias 0 -> 2
