File: Design/Sensing/sensor/kicad_simulations/sensor/sensor.kicad_sch (KiCad schematic)
At the start: 38 parts, among them J1 Conn_01x02_Pin, J10 Conn_01x02_Pin, J11 Conn_01x02_Pin, J12 Conn_01x02_Pin, J13 Conn_01x02_Pin, J14 Conn_01x01_Pin, J15 Conn_01x01_Pin, J16 Conn_01x02_Pin, J17 Conn_01x02_Pin, J2 Conn_01x02_Pin, J3 Conn_02x14_Odd_Even, J5 L_S_B, J6 Conn_01x01_Pin, J7 Conn_01x02_Pin, J8 Conn_01x02_Pin, J9 Conn_01x02_Pin, Q1 MMBT5551L, Q2 MMBT5551L, Q3 MMBT5551L, U1 LM324, U2 TSSP58038, U3 TSSP58038, U4 TSSP58038

Commit message: Updated the schematic
Connections:
- net 3V3 renamed +3.3V
Other:
- company: (none) -> University of Cape Town
- moved on the sheet: D1, D3, J10, J11, J12, J13, J14, J15, J16, J17, J8, J9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

Commit message: Libraries for demo updated
Connections:
- net PA6 renamed PA6_ADC
- net PA7 renamed PA7_ADC
- net PC4 renamed PC4_ADC
- net PE15 renamed PE15_TIM
Other:
- note added: "- Failure management circuit for the IR Receiver."
- note added: "- Failure management for the IR LED."
- note added: "- The emitter and receiver circuits are powered by a 3V3 power rail. - PE15_TIM is connected to a timing register in the uC, it is used for switching on/off the NPN transistor for power saving. - PA6_ADC(Left sensor output) is connected to the uC analog input(ADC)"
- note added: "- The emitter and receiver circuits are powered by a 3V3 power rail. - PE15_TIM is connected to a timing register in the uC, it is used for switching on/off the NPN transistor for power saving. - PA7_ADC(Left sensor output) is connected to the uC analog input(ADC)"
- note added: "- The emitter and receiver circuits are powered by a 3V3 power rail. - PE15_TIM is connected to a timing register in the uC, it is used for switching on/off the NPN transistor for power saving. - PC4_ADC(Left sensor output) is connected to the uC analog input(ADC)"
- note added: "Emitter"
- note added: "Microprocessor pinouts"
- note added: "Receiver"
- note removed: "- PA3 is used for switching on/off the NPN transistor for power saving. - It uses the internal TIM14 register to create delays and complete the timing circuitry(sleep/wake). - PA6(Left sensor output) is connected to the uC analog input"
- note removed: "- PA4 is used for switching on/off the NPN transistor for power saving. - It uses the internal TIM14 register to create delays and complete the timing circuitry(sleep/wake). - PA7(Left sensor output) is connected to the uC analog input"
- note removed: "- PA5 is used for switching on/off the NPN transistor for power saving. - It uses the internal TIM14 register to create delays and complete the timing circuitry(sleep/wake). - PC4(Left sensor output) is connected to the uC analog input"
- note removed: "INCORRECT NET PLACING, CORRECT IT USING THE PCB ONE"
- title: (none) -> Sensing Subsystem
- moved on the sheet: D1, D2, D3, J1, J10, J11, J12, J13, J14, J15, J16, J17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
