File: Design/Power/Kicad/project.kicad_sch (KiCad schematic)
At the start: 26 parts, among them IC1 TP4056-42-ESOP8, IC2 A3901SEJTR-T, J1 Pins_02x08_P1.27mm_SMT, J2 JST_02

Commit message: Add files via upload
All the KICAD FILES FOR THE PROJECT
Parts:
- IC2: Mouser Part Number 250-A3901SEJTR-T -> Motor driver
Other:
- note added: "A Slide switch that turns the system on and OFF , it does this by opening the circuit between the battery and the load"
- note added: "EP is the thermal protection for the IC"
- note added: "LED2 TURNS ON WHEN THE BATTERY IS DONE CHARGING AND NOT CHARGING LED1 TURNS ON WHEN THE BATTERY IS CHARGING"
- note added: "Load is the power supply to the motor driving IC"
- note added: "Motor 1B and Motor 1 are the terminals of the motors"
- note added: "Motor 2B and Motor 2 are the terminals of the motors"
- note added: "Motor_Driver"
- note added: "PMW1 will be controlling the speed of motor 1 PMW3 will be controlling the speed of motor 2 PMW2 will be controlling the direction of motor 1 PMW4 will be controlling the direction of motor 2"
- note added: "The ADC terminal to check the battery status"
- moved on the sheet: IC2
